File: Section A - Title A.kicad_sch (KiCad schematic)
At the start: 0 parts

Commit message: First draft
Parts:
- added D1: 16-213/SDRC/S530-A3/TR8, diodos_LED_SMD:LED_0402_1005Metric, symbol diodos_LED:16-213/SDRC/S530-A3/TR8
- added R1: RC0402FR-071KL, resistores_SMD:R_0402_1005Metric, symbol resistores:RC0402FR-071KL
Connections:
- new net: D1.2 (A), R1.2
- new net +3V0: R1.1
- new net GND: D1.1 (K)
